Commit message: Made tip the penguin beak

File: threedof/threedof_description/urdf/threedof.urdf (robot description, URDF)
Before this commit: robot threedof, 5 links, 4 joints
Links:
- added link tip_link, mass 0
Joints:
- added joint tip_joint: type fixed, parent penguin_link, child tip_link, origin xyz=0.316 0 0 rpy=0 0 0, axis 0 0 1
