Commit message: Changes from past while

File: pianoman_description/urdf/pianoman.urdf (robot description, URDF)
Before this commit: robot pianoman, 9 links, 8 joints
Links:
- added link L_tip_link, mass 0
- added link R_tip_link, mass 0
Joints:
- removed joint global_pan_joint
- added joint L_tip_joint: type fixed, parent L_upper_link, child L_tip_link, origin xyz=0.403 0 0 rpy=0 0 0, axis 0 0 1
- added joint R_tip_joint: type fixed, parent R_upper_link, child R_tip_link, origin xyz=0.403 0 0 rpy=0 0 0, axis 0 0 1
- added joint base_joint: type continuous, parent base_link, child palm_link, origin xyz=0.04 0.038 0.04375 rpy=0 0 0, axis 0 0 1
- joint L_upper_joint: origin xyz=0.25 0 -0.03105 rpy=-3.1416 0 0 -> xyz=0.25 0 0.03105 rpy=0 0 0
- joint R_lower_joint: origin xyz=-0.01505 0 0.11 rpy=3.1416 -1.5708 0 -> xyz=-0.01505 0 0.11 rpy=0 -1.5708 0
- joint R_upper_joint: origin xyz=0.25 0 -0.03105 rpy=-3.1416 4.1111E-05 0 -> xyz=0.25 0 -0.03105 rpy=0 4.1111E-05 0

Commit message: Calculating working rotation angle now and fixed inverse kinematics bug.

File: pianoman_description/urdf/pianoman.urdf (robot description, URDF)
Before this commit: robot pianoman, 11 links, 10 joints
Joints:
- joint L_tip_joint: origin xyz=0.403 0 0 rpy=0 0 0 -> xyz=0.393 0 0 rpy=0 0 0
- joint R_tip_joint: origin xyz=0.403 0 0 rpy=0 0 0 -> xyz=0.393 0 0 rpy=0 0 0

Commit message: Added secondary task to match keyboard angle.

File: pianoman_description/urdf/pianoman.urdf (robot description, URDF)
Before this commit: robot pianoman, 11 links, 10 joints
Joints:
- joint L_tip_joint: origin xyz=0.393 0 0 rpy=0 0 0 -> xyz=0.385 0 -0.015 rpy=0 0 0
- joint R_tip_joint: origin xyz=0.393 0 0 rpy=0 0 0 -> xyz=0.385 0 -0.015 rpy=0 0 0

Commit message: things work--about to optimize gains.

File: pianoman_description/urdf/pianoman.urdf (robot description, URDF)
Before this commit: robot pianoman, 11 links, 10 joints
Joints:
- joint L_tip_joint: origin xyz=0.385 0 -0.015 rpy=0 0 0 -> xyz=0.421 0 -0.015 rpy=0 0 0
- joint R_tip_joint: origin xyz=0.385 0 -0.015 rpy=0 0 0 -> xyz=0.421 0 -0.015 rpy=0 0 0

Commit message: Things are working for the most part

File: pianoman_description/urdf/pianoman.urdf (robot description, URDF)
Before this commit: robot pianoman, 11 links, 10 joints
Joints:
- joint R_tip_joint: origin xyz=0.421 0 -0.015 rpy=0 0 0 -> xyz=0.423 0 -0.015 rpy=0 0 0

Commit message: Last commit before incorporating pulling

File: pianoman_description/urdf/pianoman.urdf (robot description, URDF)
Before this commit: robot pianoman, 11 links, 10 joints
Joints:
- joint L_tip_joint: origin xyz=0.421 0 -0.015 rpy=0 0 0 -> xyz=0.421 0.005 -0.015 rpy=0 0 0
- joint R_tip_joint: origin xyz=0.423 0 -0.015 rpy=0 0 0 -> xyz=0.423 0.005 -0.015 rpy=0 0 0
